File: Erica_Polivoks_EG_Panel.kicad_pcb (KiCad board)
At the start: 2 copper layers, 40.3 x 128.5 mm, 13 parts

Commit message: v1.0 ready for production
Changed lines of the file:
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@@
 		(pad_to_mask_clearance 0)
 		(allow_soldermask_bridges_in_footprints no)
+		(grid_origin 60.07 83.3)
 		(pcbplotparams
 			(layerselection 0x0000020_7ffffffe)
@@
 		(pad "1" thru_hole circle
 			(at 0 0)
-			(size 5.969 5.969)
-			(drill 4.953)
+			(size 8 8)
+			(drill 7)
 			(layers "*.Cu" "*.Mask")
 			(remove_unused_layers no)
